File: OpenVideoModulator.sch (KiCad schematic (older format))
At the start: 22 parts, among them J1 CONN_6, J2 S-Video+Composite_Combo, P1 OSHW_LOGO, U1 AD724, Y1 4.433619M

Commit message: 1st version
Parts:
- added D1: 1N4001, Diode_SMD:D_SMA, symbol Diode:1N4001
- added J3: RCA, OpenVideoModulator:CUI_RCJ-044, symbol Connector:Conn_Coaxial
- added J4: Mini-DIN-4, OpenVideoModulator:CUI_MD-40S_1234, symbol Connector:Mini-DIN-4
- added J5: Conn_01x04_Male, Connector_PinHeader_2.54mm:PinHeader_1x04_P2.54mm_Vertical, symbol Connector:Conn_01x04_Male
- added J6: Barrel_Jack, Connector_BarrelJack:BarrelJack_Horizontal, symbol Connector:Barrel_Jack
- C10, C8, C9: footprint Capacitor_THT:CP_Radial_D6.3mm_P2.50mm -> Capacitor_THT:CP_Radial_D5.0mm_P2.00mm
- C6: footprint Capacitor_SMD:CP_Elec_6.3x5.8 -> Capacitor_THT:CP_Radial_D5.0mm_P2.00mm
- C7: footprint Capacitor_SMD:C_1206_3216Metric_Pad1.42x1.75mm_HandSolder -> Capacitor_SMD:C_0805_2012Metric_Pad1.15x1.40mm_HandSolder
- J1: symbol conn:CONN_6 -> OpenVideoModulator-rescue:CONN_6-conn
- J2: footprint (none) -> OpenVideoModulator:AV-MDC-401
- P1: symbol conn:CONN_1 -> OpenVideoModulator-rescue:CONN_1-conn
Connections:
- net labels added: COMP, CRMA, LUMA
Other:
- note added: "Combo connector"
- note added: "Separated connectors"
- moved on the sheet: C1, C10, C2, C3, C4, C8, C9, J2A, J2B, J2C, JP1, R1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

Commit message: panelizing experiments
Parts:
- J1: value CONN_6 -> CONN_7; footprint Connector_PinHeader_2.54mm:PinHeader_1x06_P2.54mm_Vertical -> Connector_PinHeader_2.54mm:PinHeader_1x07_P2.54mm_Vertical; symbol OpenVideoModulator-rescue:CONN_6-conn -> Connector:Conn_01x07_Male
Connections:
- no-connect marks 1 -> 2
Changed lines of the file:
@@
 	4710 3045 4875 3045
 $Comp
-L OpenVideoModulator-rescue:CONN_6-conn J1
+L Connector:Conn_01x07_Male J1
 U 1 1 5C9A7D83
-P 2075 1705
-F 0 "J1" H 1944 2192 60  0000 C CNN
-F 1 "CONN_6" H 1944 2086 60  0000 C CNN
-F 2 "Connector_PinHeader_2.54mm:PinHeader_1x06_P2.54mm_Vertical" H 2075 1705 50  0001 C CNN
-F 3 "" H 2075 1705 50  0001 C CNN
-	1    2075 1705
-	-1   0    0    -1
-$EndComp
-Wire Wire Line
-	2425 1455 2525 1455
-Wire Wire Line
-	2425 1555 2525 1555
+P 2225 1655
+F 0 "J1" H 2094 2142 60  0000 C CNN
+F 1 "CONN_7" H 2094 2036 60  0000 C CNN
+F 2 "Connector_PinHeader_2.54mm:PinHeader_1x07_P2.54mm_Vertical" H 2225 1655 50  0001 C CNN
+F 3 "" H 2225 1655 50  0001 C CNN
+	1    2225 1655
+	1    0    0    -1
+$EndComp
 $Comp
 L power:VCC #PWR015
@@
 	1    0    0    -1
 $EndComp
-Wire Wire Line
-	2525 1335 2525 1455
-Wire Wire Line
-	2525 1555 2525 2050
 $Comp
 L power:GND #PWR016
@@
 	1    0    0    -1
 $EndComp
-Text Label 2585 1655 0    50   ~ 0
+Text Label 2570 1955 0    50   ~ 0
 sync_in
-Text Label 2585 1755 0    50   ~ 0
+Text Label 2575 1855 0    50   ~ 0
 red_in
-Text Label 2585 1855 0    50   ~ 0
+Text Label 2570 1755 0    50   ~ 0
 green_in
-Text Label 2585 1955 0    50   ~ 0
+Text Label 2565 1655 0    50   ~ 0
 blue_in
 Wire Wire Line
@@
 L power:GND #PWR0112
 U 1 1 60610F39
-P 8400 1890
-F 0 "#PWR0112" H 8400 1640 50  0001 C CNN
-F 1 "GND" V 8405 1762 50  0000 R CNN
-F 2 "" H 8400 1890 50  0001 C CNN
-F 3 "" H 8400 1890 50  0001 C CNN
-	1    8400 1890
+P 8400 1590
+F 0 "#PWR0112" H 8400 1340 50  0001 C CNN
+F 1 "GND" V 8405 1462 50  0000 R CNN
+F 2 "" H 8400 1590 50  0001 C CNN
+F 3 "" H 8400 1590 50  0001 C CNN
+	1    8400 1590
 	0    -1   -1   0
 $EndComp
+Text GLabel 8400 1790 2    50   Input ~ 0
+CRMA
+Text GLabel 8400 1890 2    50   Input ~ 0
+LUMA
 Text GLabel 8400 1690 2    50   Input ~ 0
-CRMA
-Text GLabel 8400 1790 2    50   Input ~ 0
-LUMA
-Text GLabel 8400 1590 2    50   Input ~ 0
 COMP
 $Comp
@@
 Wire Wire Line
 	2500 2825 2660 2825
+Wire Wire Line
+	2525 1335 2525 1355
+Wire Wire Line
+	2525 1355 2425 1355
+NoConn ~ 2430 1555
+Wire Wire Line
+	2525 2050 2525 1455
+Wire Wire Line
+	2525 1455 2425 1455
 $EndSCHEMATC

Commit message: release candidate
Parts:
- removed J2: S-Video+Composite_Combo, OpenVideoModulator:AV-MDC-401, symbol s-video+composite_combo:S-Video+Composite_Combo
- added H1, H2: MountingHole, MountingHole:MountingHole_2.2mm_M2_ISO7380_Pad, symbol Mechanical:MountingHole
- JP1: footprint OpenVideoModulator:SolderJumper-3_P1.3mm_Bridged12_RoundedPad1.0x1.5mm -> Connector_PinHeader_2.54mm:PinHeader_1x03_P2.54mm_Vertical
Connections:
- wire segments 115 -> 105
Other:
- note added: "5V input connectors"
- note added: "Mounting holes"
- note added: "RGBS Input"
- note added: "Separated video connectors"
- note removed: "Combo connector"
- moved on the sheet: C1, C10, C2, C3, C4, C8, C9, D1, J1, J3, J4, J5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
